Commit message: actualitzacio week_3

File: urdf/week_2.urdf (robot description, URDF)
Before this commit: robot week_2, 9 links, 8 joints
Links:
- link omniwheel: geometry visual mesh filename=package://robot/meshes/omniwheel.stl
- link rodeta_1: geometry visual mesh filename=package://robot/meshes/rodeta.stl
- link rodeta_2: geometry visual mesh filename=package://robot/meshes/rodeta.stl
- link rodeta_3: geometry visual mesh filename=package://robot/meshes/rodeta.stl
- link rodeta_4: geometry visual mesh filename=package://robot/meshes/rodeta.stl
- link rodeta_5: geometry visual mesh filename=package://robot/meshes/rodeta.stl
- link rodeta_6: geometry visual mesh filename=package://robot/meshes/rodeta.stl
- link rodeta_7: geometry visual mesh filename=package://robot/meshes/rodeta.stl
- link rodeta_8: geometry visual mesh filename=package://robot/meshes/rodeta.stl
