Commit message: actualitzat 17/10/17

File: urdf/week_4.urdf (robot description, URDF)
Before this commit: robot robot, 1 links, 0 joints
Links:
- added link bottom_propeller, mass 0.0078; collision cylinder length=0.05 radius=0.0125; visual mesh filename=package://robot/meshes/bottom_propeller.stl
- added link fake_link; collision cylinder length=0.05 radius=0.01; visual cylinder length=0.05 radius=0.01
- added link motor_frame, mass 0.097; collision cylinder length=0.2 radius=0.225; visual mesh filename=package://robot/meshes/plat_superior.stl
- added link top_propeller, mass 0.0078; collision cylinder length=0.05 radius=0.0125; visual mesh filename=package://robot/meshes/top_propeller.stl
- link base: geometry collision cylinder length=0.11 radius=0.225; visual mesh filename=package://robot/meshes/main_body.stl scale=0.001 0.001 0.001
Joints:
- added joint bottom_propeller: type continuous, parent motor_frame, child bottom_propeller, origin xyz=0 0 0 rpy=0 0 0, axis 0 0 1
- added joint rev1: type revolute, parent base, child fake_link, origin xyz=0 0 0.005432 rpy=0 0 ${90*pi/180}, axis 1 0 0, limit lower=${-45*pi/180} upper=${45*pi/180} effort=100000 velocity=${2*pi}
- added joint rev2: type revolute, parent fake_link, child motor_frame, origin xyz=0 0 0 rpy=0 0 1 , axis 1 0 0, limit lower=${-45*pi/180} upper=${45*pi/180} effort=100000. velocity=${2*pi}
- added joint top_propeller: type continuous, parent motor_frame, child top_propeller, origin xyz=0 0 0 rpy=0 0 0, axis 0 0 1

Commit message: actualitzacio 17/10/22

File: urdf/week_4.urdf (robot description, URDF)
Before this commit: robot robot, 5 links, 4 joints
Links:
- link fake_link: mass None -> 0.015
