Commit message: actualitzacio moments inercia

File: urdf/week_5.urdf (robot description, URDF)
Before this commit: robot robot, 5 links, 4 joints
Links:
- link bottom_propeller: geometry collision cylinder length=0.01 radius=0.125; visual mesh filename=package://robot/meshes/bottom_propeller_0_0_0.stl
- link fake_link: mass 0.015 -> 0.000014; geometry collision mesh filename=package://robot/meshes/fake_0_0.stl; visual mesh filename=package://robot/meshes/fake_0_0.stl
- link motor_frame: mass 0.097 -> 0.094; geometry collision cylinder length=0.035 radius=0.125; visual mesh filename=package://robot/meshes/plat_superior_0_0_0.stl
- link top_propeller: geometry collision cylinder length=0.01 radius=0.125; visual mesh filename=package://robot/meshes/top_propeller_0_0_0.stl
Joints:
- joint rev1: limit lower=${-45*pi/180} upper=${45*pi/180} effort=100000 velocity=${2*pi} -> lower=${-35*pi/180} upper=${35*pi/180} effort=100000 velocity=${2*pi}; origin xyz=0 0 0.005432 rpy=0 0 ${90*pi/180} -> xyz=0 0 0.07024 rpy=0 0 ${90*pi/180}
- joint rev2: axis 1 0 0 -> 0 1 0; limit lower=${-45*pi/180} upper=${45*pi/180} effort=100000. velocity=${2*pi} -> lower=${-35*pi/180} upper=${35*pi/180} effort=100000. velocity=${2*pi}

Commit message: actualització 17/12/02

File: urdf/week_5.urdf (robot description, URDF)
Before this commit: robot robot, 5 links, 4 joints
Links:
- link fake_link: mass 0.000014 -> 0.000510
- link motor_frame: mass 0.094 -> 0.0679
