Commit message: actualitzacio previa presentacio

File: urdf/week_6.urdf (robot description, URDF)
Before this commit: robot robot, 5 links, 4 joints
Links:
- link base: mass 0.42 -> 0.1; geometry collision cylinder length=0.05 radius=0.1; visual mesh filename=package://robot/meshes/main_body.stl scale=0.001 0.001 0.001
- link fake_link: mass 0.000510 -> 0.0679
Joints:
- joint bottom_propeller: limit effort=999999 velocity=${1000*pi} -> effort=999999 velocity=50000
- joint rev2: origin xyz=0 0 0 rpy=0 0 1  -> xyz=0 0 0 rpy=0 0 0 
- joint top_propeller: limit effort=999999 velocity=${1000*pi} -> effort=999999 velocity=50000
