Commit message: brac i suport

File: urdf/spm_1.urdf (robot description, URDF)
Before this commit: robot spm_1, 6 links, 5 joints
Links:
- removed link fork
- added link axis_arm_2; visual cylinder length=0.01 radius=0.002
- added link plat_superior; visual mesh filename=package://robot/meshes/plat_superior.stl scale=0.001 0.001 0.001
Joints:
- removed joint rev_3
- added joint arm_2_to axis_arm_2: type fixed, parent arm_2, child axis_arm_2, origin xyz=0 -0.05327 -0.01067 rpy=${202.5*pi/180} 0 0, axis 0 0 1
- added joint plat_superior_joint: type fixed, parent axis_arm_2, child plat_superior, origin xyz=0 0 0.13855 rpy=${247.5*pi/180} 0 0, axis 0 1 0 

Commit message: monents inercia i collissio

File: urdf/spm_1.urdf (robot description, URDF)
Before this commit: robot spm_1, 7 links, 6 joints
Links:
- removed link arm_1
- removed link arm_2
- removed link axis_arm_2
- removed link base
- removed link motor_axis
- removed link stepper_motor
- link plat_superior: mass None -> 0.0679; geometry collision cylinder length=0.050 radius=0.125; visual mesh filename=package://robot/meshes/plat_superior.stl scale=0.001 0.001 0.001
Joints:
- removed joint arm_2_to axis_arm_2
- removed joint base_to_stepper_motor
- removed joint motor_to_axis
- removed joint rev_1
- removed joint rev_2

File: urdf/spm_2.urdf (robot description, URDF)
Before this commit: robot spm_1, 1 links, 0 joints
Links:
- removed link fake_1
- added link arm_1, mass 0.02; collision mesh filename=package://robot/meshes/inferior_arm.stl scale=0.001 0.001 0.001; visual mesh filename=package://robot/meshes/inferior_arm.stl scale=0.001 0.001 0.001
- added link arm_2, mass 0.008; collision mesh filename=package://robot/meshes/as.stl scale=0.001 0.001 0.001; visual mesh filename=package://robot/meshes/as.stl scale=0.001 0.001 0.001
- added link axis_arm_2, mass 0.010; collision cylinder length=0.01 radius=0.0015; visual cylinder length=0.01 radius=0.002
- added link base
- added link motor_axis, mass 0.010; collision cylinder length=0.01 radius=0.0015; visual mesh filename=package://robot/meshes/eix_motor.stl scale=0.001 0.001 0.001
- added link plat_superior, mass 0.0679; collision cylinder length=0.050 radius=0.125; visual mesh filename=package://robot/meshes/plat_superior.stl scale=0.001 0.001 0.001
- added link stepper_motor, mass 0.1; collision cylinder length=0.034 radius=0.016; visual mesh filename=package://robot/meshes/motor.stl scale=0.001 0.001 0.001
Joints:
- added joint arm_2_to axis_arm_2: type fixed, parent arm_2, child axis_arm_2, origin xyz=0 -0.05327 -0.01067 rpy=${202.5*pi/180} 0 0, axis 0 0 1
- added joint base_to_stepper_motor: type fixed, parent base, child stepper_motor, origin xyz=0 0 0 rpy=0 0 0, axis 0 0 1
- added joint motor_to_axis: type fixed, parent stepper_motor, child motor_axis, origin xyz=0 0.12926 0.06335 rpy=${-112.5*pi/180} 0 0, axis 0 0 1
- added joint plat_superior_joint: type fixed, parent axis_arm_2, child plat_superior, origin xyz=0 0 0.13855 rpy=${247.5*pi/180} 0 0, axis 0 1 0 
- added joint rev_1: type revolute, parent motor_axis, child arm_1, origin xyz=0 0 0 rpy=0 0 0, axis 0 0 1, limit lower=${-45*pi/180} upper=${45*pi/180} effort=100000 velocity=${2*pi}
- added joint rev_2: type revolute, parent arm_1, child arm_2, origin xyz=0 -0.05327 -0.01067 rpy=${22.5*pi/180} 0 0, axis 0 0 1, limit lower=${-45*pi/180} upper=${45*pi/180} effort=100000 velocity=${2*pi}
