Commit message: actualitzacio_week_3

File: urdf/week_3.urdf (robot description, URDF)
Before this commit: robot week_3, 5 links, 4 joints
Links:
- removed link fake_link
- removed link helix1
- removed link helix2
- removed link motor_frame
Joints:
- removed joint motor1
- removed joint motor2
- removed joint rev1
- removed joint rev2

Commit message: actualitzacio 170924

File: urdf/week_3.urdf (robot description, URDF)
Before this commit: robot week_3, 1 links, 0 joints
Links:
- added link bottom_propeller, mass 0.0078; collision cylinder length=0.05 radius=0.0125; visual mesh filename=package://robot/meshes/bottom_propeller.stl
- added link fake_link; collision cylinder length=0.05 radius=0.01; visual cylinder length=0.05 radius=0.01
- added link motor_frame; visual mesh filename=package://robot/meshes/plat_superior.stl
- added link top_propeller, mass 0.0078; collision cylinder length=0.05 radius=0.0125; visual mesh filename=package://robot/meshes/top_propeller.stl
Joints:
- added joint bottom_propeller: type continuous, parent motor_frame, child bottom_propeller, origin xyz=0 0 0 rpy=0 0 0, axis 0 0 1
- added joint rev1: type revolute, parent base, child fake_link, origin xyz=0 0 0.005432 rpy=0 0 ${90*pi/180}, axis 1 0 0, limit lower=${-45*pi/180} upper=${45*pi/180} effort=100000 velocity=${2*pi}
- added joint rev2: type revolute, parent fake_link, child motor_frame, origin xyz=0 0 0 rpy=0 0 1 , axis 1 0 0, limit lower=${-45*pi/180} upper=${45*pi/180} effort=100000. velocity=${2*pi}
- added joint top_propeller: type continuous, parent motor_frame, child top_propeller, origin xyz=0 0 0 rpy=0 0 0, axis 0 0 1

Commit message: urdf xacro definida

File: urdf/week_3.urdf (robot description, URDF)
Before this commit: robot week_3, 5 links, 4 joints
Links:
- removed link bottom_propeller
- removed link fake_link
- removed link motor_frame
- removed link top_propeller
Joints:
- removed joint bottom_propeller
- removed joint rev1
- removed joint rev2
- removed joint top_propeller
